File: usb_push_sw.sch (KiCad schematic (older format))
At the start: 7 parts

Commit message: とりあえず引いた ERC OK
Parts:
- removed U? (x3): SW_push_2pin, symbol kicad_mylib:SW_push_2pin
- added SW1, SW2, SW3: SW_Push_Open_Dual, symbol Switch:SW_Push_Open_Dual
- gave numbers to parts that had none: 4
Connections:
- net +3V3: now also U1.12 (3V3), SW1.1, SW2.1, SW3.1; no longer U1.1 (PA02_A0_D0), U1.2 (PA4_A1_D1), U1.3 (PA10_A2_D2)
- net GND: now also U1.13 (GND)
- net at R1.1: now also U1.1 (PA02_A0_D0), SW1.2
- net at R2.1: now also U1.2 (PA4_A1_D1), SW2.2
- net at R3.1: now also U1.3 (PA10_A2_D2), SW3.2
- no-connect marks 0 -> 15
Other:
- moved on the sheet: R1, R2, R3, U1
